File: Hardware/DE0_Digital_IO_Wing.brd (EAGLE design)
At the start: 111.8 x 57.1 mm, 22 parts, among them J1 929975-01-20-RK, J2 929975-01-20-RK, U1 SN74LVC8T245PWR, U2 SN74LVC8T245PWR, U3 SN74LVC8T245PWR, U4 SN74LVC8T245PWR

Commit message: Fixed weird missing trace from Pin3 U1
Connections:
- net GPIO0_D14: now also U1.P$3
Routing:
- net GPIO0_D14: track 110.7 -> 112.4 mm
Changed lines of the file:
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@@
 <wire x1="93.227753125" y1="28.194" x2="96.446284375" y2="28.194" width="0.254" layer="1"/>
 <wire x1="96.446284375" y1="28.194" x2="100.573" y2="24.067284375" width="0.254" layer="1"/>
+<contactref element="U1" pad="P$3"/>
+<wire x1="100.573" y1="24.067284375" x2="100.573" y2="22.358" width="0.254" layer="1"/>
 </signal>
 <signal name="GPIO0_D15">
