File: Hardware/DE0_Digital_IO_Wing.brd (EAGLE design)
At the start: 111.8 x 57.1 mm, 22 parts, among them J1 929975-01-20-RK, J2 929975-01-20-RK, U1 SN74LVC8T245PWR, U2 SN74LVC8T245PWR, U3 SN74LVC8T245PWR, U4 SN74LVC8T245PWR

Commit message: Bringing it to current library spec.
Parts:
- J1, J2: device PP_Connectors:HEADER_02X20_PTH -> PP_Connectors:2.54MM_02X20_PIN_HEADER
- U1, U2, U3, U4: device PP_DigitalIC:TTSOP-24 -> PP_DigitalIC:SN74LVC8T245_TTSOP-24
