File: Hardware/DE0_Digital_IO_Wing.sch (EAGLE design)
At the start: 22 parts, among them J1 929975-01-20-RK, J2 929975-01-20-RK, U1 SN74LVC8T245PWR, U2 SN74LVC8T245PWR, U3 SN74LVC8T245PWR, U4 SN74LVC8T245PWR

Commit message: Bringing it to current library spec.
Parts:
- AUX_POWER: device PP_Connectors:PH_1X04282834-4 -> PP_Connectors:CON_01X04_282834-4; LABEL00 3.3V -> (none); LABEL01 GND -> 3.3V; LABEL02 5V -> GND; LABEL03 GND -> 5V; LABEL04 (none) -> GND
- J1, J2: device PP_Connectors:PH_2X20HEADER_02X20_PTH -> PP_Connectors:CON_02X202.54MM_PIN_HEADER
Other:
- moved on the sheet: J1, J2, U1, U2, U3, U4
